File: KiCad/LeChiffre.kicad_pcb (KiCad board)
At the start: 2 copper layers, 228.4 x 85 mm, 105 parts, among them J1 Conn_01x03_Female, J2 Conn_01x04_Female, SW1 SW_Push, SW10 SW_Push, SW11 SW_Push, SW12 SW_Push, SW13 SW_Push, SW14 SW_Push, SW15 SW_Push, SW16 SW_Push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

Commit message: Update PCB
Routing:
- net Net-(D105-Pad2): track 64.9 -> 65.7 mm
- net Net-(D107-Pad2): track 51.8 -> 52.4 mm
