File: KiCad/Le Chiffre v2/LeChiffre_Plate/LeChiffre_Plate.kicad_pcb (KiCad board)
At the start: 2 copper layers, 107.1 x 92.5 mm, 1 part, among them J1 Conn_01x01_Female

Commit message: Adding BOM and Gerber files
Other:
- board text removed: "JLCJLCJLCJLC"
Changed lines of the file:
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@@
-(kicad_pcb (version 20171130) (host pcbnew "(5.1.2-1)-1")
+(kicad_pcb (version 20171130) (host pcbnew "(5.1.10-1-10_14)")
   (general
     (thickness 1.6)
-    (drawings 188)
+    (drawings 187)
     (tracks 1)
     (zones 0)
@@
       (effects (font (size 1 1) (thickness 0.15)))
     )
+    (fp_line (start -0.7 -0.7) (end 0.7 -0.7) (layer F.SilkS) (width 0.12))
+    (fp_line (start 0.7 -0.7) (end 0.7 0.7) (layer F.SilkS) (width 0.12))
+    (fp_line (start 0.7 0.7) (end -0.7 0.7) (layer F.SilkS) (width 0.12))
+    (fp_line (start -0.7 0.7) (end -0.7 -0.7) (layer F.SilkS) (width 0.12))
+    (fp_line (start -1 -1) (end 1 -1) (layer F.CrtYd) (width 0.05))
+    (fp_line (start -1 -1) (end -1 1) (layer F.CrtYd) (width 0.05))
+    (fp_line (start 1 1) (end 1 -1) (layer F.CrtYd) (width 0.05))
     (fp_line (start 1 1) (end -1 1) (layer F.CrtYd) (width 0.05))
-    (fp_line (start 1 1) (end 1 -1) (layer F.CrtYd) (width 0.05))
-    (fp_line (start -1 -1) (end -1 1) (layer F.CrtYd) (width 0.05))
-    (fp_line (start -1 -1) (end 1 -1) (layer F.CrtYd) (width 0.05))
-    (fp_line (start -0.7 0.7) (end -0.7 -0.7) (layer F.SilkS) (width 0.12))
-    (fp_line (start 0.7 0.7) (end -0.7 0.7) (layer F.SilkS) (width 0.12))
-    (fp_line (start 0.7 -0.7) (end 0.7 0.7) (layer F.SilkS) (width 0.12))
-    (fp_line (start -0.7 -0.7) (end 0.7 -0.7) (layer F.SilkS) (width 0.12))
     (fp_text user %R (at 0 -1.45) (layer F.Fab)
       (effects (font (size 1 1) (thickness 0.15)))
@@
       (net 1 GND))
   )
-  (gr_text " JLCJLCJLCJLC" (at 185.06 131.28 -3) (layer B.SilkS)
-    (effects (font (size 1.5 1.5) (thickness 0.3)) (justify mirror))
-  )
   (gr_line (start 153.029387 137.725856) (end 135.65983 135.593142) (layer Edge.Cuts) (width 0.2))
